File: PCB/pcb-illuminator.kicad_pcb (KiCad board)
At the start: 2 copper layers, 100 x 92.5 mm, 31 parts, among them J1 USB C, J2 +5V GND, J3 from microcontroller, J4 Barrel_Jack +5V, Q1 BD433, SW1 on/off

Commit message: move connectors, add another led row
Parts:
- removed J1: USB C, Connector_USB:USB_C_Receptacle_GCT_USB4085
- removed the REF** at (158.0, 143.0)
- removed the REF** at (112.0, 142.5)
- removed the REF** at (112.5, 84.0)
- removed the REF** at (160.5, 85.5)
- added D10: LED, LED_THT:LED_D5.0mm, F.Cu at (157.0, 135.0)
- added D11: LED, LED_THT:LED_D5.0mm, F.Cu at (135.0, 135.0)
- added D12: LED, LED_THT:LED_D5.0mm, F.Cu at (110.0, 135.0)
- added R5: 14 ohm 2W, Resistor_THT:R_Axial_DIN0411_L9.9mm_D3.6mm_P15.24mm_Horizontal, F.Cu at (190.0, 124.0)
- added REF**: MountingHole_3.2mm_M3_DIN965, MountingHole:MountingHole_3.2mm_M3_DIN965, F.Cu at (159.0, 144.0)
- added REF**: MountingHole_3.2mm_M3_DIN965, MountingHole:MountingHole_3.2mm_M3_DIN965, F.Cu at (111.0, 143.0)
- added REF**: MountingHole_3.2mm_M3_DIN965, MountingHole:MountingHole_3.2mm_M3_DIN965, F.Cu at (111.0, 83.0)
- added REF**: MountingHole_3.2mm_M3_DIN965, MountingHole:MountingHole_3.2mm_M3_DIN965, F.Cu at (161.0, 84.0)
- Q1: value BD433 -> BD437
- R1, R2, R3: footprint Resistor_THT:R_Axial_DIN0309_L9.0mm_D3.2mm_P5.08mm_Vertical -> Resistor_THT:R_Axial_DIN0411_L9.9mm_D3.6mm_P15.24mm_Horizontal
- R4: footprint Resistor_THT:R_Axial_DIN0309_L9.0mm_D3.2mm_P5.08mm_Vertical -> Resistor_THT:R_Axial_DIN0309_L9.0mm_D3.2mm_P12.70mm_Horizontal
- moved R1 16.8 mm to (190.0, 116.0)
- moved R2 11.4 mm to (190.0, 108.0)
- moved R3 10.2 mm to (190.0, 100.0)
- moved D1 8.73 mm to (158.0, 121.0)
- moved D7 8.63 mm to (110.0, 121.0)
- moved D4 8.51 mm to (135.0, 121.0)
- moved D2 7.76 mm to (158.0, 106.0)
- moved D8 7.65 mm to (110.0, 106.0)
- moved D5 7.52 mm to (135.0, 106.0)
- moved D3 6.32 mm to (158.0, 92.0)
- moved D9 6.18 mm to (110.0, 92.0)
- moved D6 6.02 mm to (135.0, 92.0)
- moved R4 5.70 mm to (117.0, 76.0)
Routing:
- net Net-(D12-Pad1): track 81.8 -> 107.4 mm
- net Net-(D11-Pad1): track 0.00 -> 22.5 mm
- net Net-(D10-Pad2): track 0.00 -> 19.8 mm
- net Net-(D10-Pad1): track 0.00 -> 19.5 mm
- net GND: track 9.15 -> 0.00 mm
- net Net-(J1-PadA4): track 8.00 -> 0.00 mm
- net Net-(D3-Pad2): track 12.4 -> 18.3 mm
- net Net-(D1-Pad2): track 12.4 -> 16.3 mm
- net Net-(R1-Pad1): track 108.0 -> 111.8 mm
- net Net-(Q1-Pad3): track 7.24 -> 10.5 mm
- net Net-(D2-Pad2): track 12.4 -> 15.4 mm
- net Net-(D3-Pad1): track 23.0 -> 20.5 mm
- net Net-(D2-Pad1): track 23.0 -> 20.5 mm
- net Net-(D1-Pad1): track 23.0 -> 20.5 mm
- net +5V: track 2.08 -> 0.00 mm, vias 1 -> 0
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Other:
- board text added: "Petridish illuminator V0.2 By Chagas AM 20200917 CERN OHL-S"
- board text removed: "Petridish illuminator V0.1 By Chagas AM 20200806 CERN OHL-S"
