File: PCB/pcb-illuminator.sch (KiCad schematic (older format))
At the start: 21 parts, among them J1 USB C, J2 +5V GND, J3 from microcontroller, J4 Barrel_Jack +5V, Q1 BD433, SW1 on/off

Commit message: move connectors, add another led row
Parts:
- removed J1: USB C, Connector_USB:USB_C_Receptacle_GCT_USB4085, symbol Connector:USB_C_Receptacle_USB2.0
- added D10, D11, D12: LED, LED_THT:LED_D5.0mm, symbol Device:LED
- added R5: 14 ohm 2W, Resistor_THT:R_Axial_DIN0411_L9.9mm_D3.6mm_P15.24mm_Horizontal, symbol Device:R_Small
- Q1: value BD433 -> BD437
- R1, R2, R3: footprint Resistor_THT:R_Axial_DIN0309_L9.0mm_D3.2mm_P5.08mm_Vertical -> Resistor_THT:R_Axial_DIN0411_L9.9mm_D3.6mm_P15.24mm_Horizontal
- R4: footprint Resistor_THT:R_Axial_DIN0309_L9.0mm_D3.2mm_P5.08mm_Vertical -> Resistor_THT:R_Axial_DIN0309_L9.0mm_D3.2mm_P12.70mm_Horizontal
Connections:
- wire segments 43 -> 47
- no-connect marks 8 -> 0
Changed lines of the file:
@@
 F 0 "R3" V 3446 2450 50  0000 C CNN
 F 1 "14 ohm 2W" V 3355 2450 50  0000 C CNN
-F 2 "Resistor_THT:R_Axial_DIN0309_L9.0mm_D3.2mm_P5.08mm_Vertical" H 3250 2450 50  0001 C CNN
+F 2 "Resistor_THT:R_Axial_DIN0411_L9.9mm_D3.6mm_P15.24mm_Horizontal" H 3250 2450 50  0001 C CNN
 F 3 "~" H 3250 2450 50  0001 C CNN
 	1    3250 2450
@@
 P 5550 2100
 F 0 "Q1" V 5879 2100 50  0000 C CNN
-F 1 "BD433" V 5788 2100 50  0000 C CNN
+F 1 "BD437" V 5788 2100 50  0000 C CNN
 F 2 "Package_TO_SOT_THT:TO-126-3_Vertical" H 5750 2025 50  0001 L CIN
 F 3 "http://www.cdil.com/datasheets/bd433_42.pdf" H 5550 2100 50  0001 L CNN
@@
 F 0 "R4" H 5609 2546 50  0000 L CNN
 F 1 "270" H 5609 2455 50  0000 L CNN
-F 2 "Resistor_THT:R_Axial_DIN0309_L9.0mm_D3.2mm_P5.08mm_Vertical" H 5550 2500 50  0001 C CNN
+F 2 "Resistor_THT:R_Axial_DIN0309_L9.0mm_D3.2mm_P12.70mm_Horizontal" H 5550 2500 50  0001 C CNN
 F 3 "~" H 5550 2500 50  0001 C CNN
 	1    5550 2500
@@
 F 0 "R1" V 3446 1550 50  0000 C CNN
 F 1 "14 ohm 2W" V 3355 1550 50  0000 C CNN
-F 2 "Resistor_THT:R_Axial_DIN0309_L9.0mm_D3.2mm_P5.08mm_Vertical" H 3250 1550 50  0001 C CNN
+F 2 "Resistor_THT:R_Axial_DIN0411_L9.9mm_D3.6mm_P15.24mm_Horizontal" H 3250 1550 50  0001 C CNN
 F 3 "~" H 3250 1550 50  0001 C CNN
 	1    3250 1550
@@
 F 0 "R2" V 3446 2000 50  0000 C CNN
 F 1 "14 ohm 2W" V 3355 2000 50  0000 C CNN
-F 2 "Resistor_THT:R_Axial_DIN0309_L9.0mm_D3.2mm_P5.08mm_Vertical" H 3250 2000 50  0001 C CNN
+F 2 "Resistor_THT:R_Axial_DIN0411_L9.9mm_D3.6mm_P15.24mm_Horizontal" H 3250 2000 50  0001 C CNN
 F 3 "~" H 3250 2000 50  0001 C CNN
 	1    3250 2000
@@
 	-1   0    0    1
 $EndComp
-NoConn ~ 2000 2450
-NoConn ~ 2000 2750
-NoConn ~ 2000 2950
-NoConn ~ 2000 3050
-NoConn ~ 2000 3150
-NoConn ~ 2000 3250
-NoConn ~ 2000 3550
-NoConn ~ 2000 3650
-$Comp
-L Connector:USB_C_Receptacle_USB2.0 J1
-U 1 1 5F345DAF
-P 1400 3050
-F 0 "J1" H 1507 3917 50  0000 C CNN
-F 1 "USB C" H 1507 3826 50  0000 C CNN
-F 2 "Connector_USB:USB_C_Receptacle_GCT_USB4085" H 1550 3050 50  0001 C CNN
-F 3 "https://www.usb.org/sites/default/files/documents/usb_type-c.zip" H 1550 3050 50  0001 C CNN
-	1    1400 3050
-	1    0    0    -1
-$EndComp
-Wire Wire Line
-	1400 3950 1250 3950
-$Comp
-L power:GND #PWR01
-U 1 1 5F34C6ED
-P 1250 3950
-F 0 "#PWR01" H 1250 3700 50  0001 C CNN
-F 1 "GND" H 1255 3777 50  0000 C CNN
-F 2 "" H 1250 3950 50  0001 C CNN
-F 3 "" H 1250 3950 50  0001 C CNN
-	1    1250 3950
-	1    0    0    -1
-$EndComp
-Connection ~ 1250 3950
-Wire Wire Line
-	1250 3950 1100 3950
-$Comp
-L power:+5V #PWR04
-U 1 1 5F34CCCC
-P 2150 2650
-F 0 "#PWR04" H 2150 2500 50  0001 C CNN
-F 1 "+5V" V 2165 2778 50  0000 L CNN
-F 2 "" H 2150 2650 50  0001 C CNN
-F 3 "" H 2150 2650 50  0001 C CNN
-	1    2150 2650
-	0    1    1    0
-$EndComp
-Wire Wire Line
-	2150 2650 2000 2650
 $Comp
 L power:+5V #PWR03
@@
 Wire Wire Line
 	2850 2100 2850 2400
+$Comp
+L Device:R_Small R5
+U 1 1 5F645D6A
+P 3250 1200
+F 0 "R5" V 3446 1200 50  0000 C CNN
+F 1 "14 ohm 2W" V 3355 1200 50  0000 C CNN
+F 2 "Resistor_THT:R_Axial_DIN0411_L9.9mm_D3.6mm_P15.24mm_Horizontal" H 3250 1200 50  0001 C CNN
+F 3 "~" H 3250 1200 50  0001 C CNN
+	1    3250 1200
+	0    -1   -1   0
+$EndComp
+Wire Wire Line
+	2850 1550 2850 1200
+Wire Wire Line
+	2850 1200 3150 1200
+Connection ~ 2850 1550
+$Comp
+L Device:LED D10
+U 1 1 5F6470D7
+P 3700 1200
+F 0 "D10" H 3693 945 50  0000 C CNN
+F 1 "LED" H 3693 1036 50  0000 C CNN
+F 2 "LED_THT:LED_D5.0mm" H 3700 1200 50  0001 C CNN
+F 3 "~" H 3700 1200 50  0001 C CNN
+	1    3700 1200
+	-1   0    0    1
+$EndComp
+$Comp
+L Device:LED D11
+U 1 1 5F647634
+P 4200 1200
+F 0 "D11" H 4193 945 50  0000 C CNN
+F 1 "LED" H 4193 1036 50  0000 C CNN
+F 2 "LED_THT:LED_D5.0mm" H 4200 1200 50  0001 C CNN
+F 3 "~" H 4200 1200 50  0001 C CNN
+	1    4200 1200
+	-1   0    0    1
+$EndComp
+$Comp
+L Device:LED D12
+U 1 1 5F647C3F
+P 4700 1200
+F 0 "D12" H 4693 945 50  0000 C CNN
+F 1 "LED" H 4693 1036 50  0000 C CNN
+F 2 "LED_THT:LED_D5.0mm" H 4700 1200 50  0001 C CNN
+F 3 "~" H 4700 1200 50  0001 C CNN
+	1    4700 1200
+	-1   0    0    1
+$EndComp
+Wire Wire Line
+	3350 1200 3550 1200
+Wire Wire Line
+	3850 1200 4050 1200
+Wire Wire Line
+	4350 1200 4550 1200
+Wire Wire Line
+	4850 1200 5050 1200
+Wire Wire Line
+	5050 1200 5050 1550
+Connection ~ 5050 1550
 $EndSCHEMATC
